Commit message: wheel1などの変数の変更

File: src/simc/urdf/common.xacro (robot description, xacro)
@@ -60,8 +60,8 @@
       <type>transmission_interface/SimpleTransmission</type>
       <joint name="${base_joint_name}">
-  <hardwareInterface>PositionJointInterface</hardwareInterface>
+  <hardwareInterface>hardware_interface/PositionJointInterface</hardwareInterface>
       </joint>
    <actuator name="${base_joint_name}_motor">
-  <hardwareInterface>PositionJointInterface</hardwareInterface>
+  <hardwareInterface>hardware_interface/PositionJointInterface</hardwareInterface>
   <mechanicalReduction>100</mechanicalReduction>
       </actuator>
@@ -70,8 +70,8 @@
       <type>transmission_interface/SimpleTransmission</type>
       <joint name="${wheel_name}_joint">
-  <hardwareInterface>VelocityJointInterface</hardwareInterface>
+  <hardwareInterface>hardware_interface/VelocityJointInterface</hardwareInterface>
       </joint>
    <actuator name="${wheel_name}_motor">
-  <hardwareInterface>VelocityJointInterface</hardwareInterface>
+  <hardwareInterface>hardware_interface/VelocityJointInterface</hardwareInterface>
   <mechanicalReduction>100</mechanicalReduction>
       </actuator>

File: src/simc/urdf/my_robo.xacro (robot description, xacro)
@@ -7,53 +7,53 @@
     <box_create mass="10" height="0.1" width="0.8" depth="0.8"/>
  </link>
-<unit_create base_name="base_wheel1_link" wheel_name="wheel1"/>
-  <joint name="base_joint1" type="continuous">
-    <parent link="base_link"/>
-    <child link="base_wheel1_link"/>
+<unit_create base_name="left_front_steering" wheel_name="left_front_wheel"/>
+  <joint name="left_front_steering_joint" type="continuous">
+    <parent link="base_link"/>
+    <child link="left_front_steering"/>
     <origin rpy="0 0 0" xyz="0.35 0.35 -0.055"/>
     <axis xyz="0 0 1"/>
   </joint>
-  <joint name="wheel1_joint" type="continuous">
-    <parent link="base_wheel1_link"/>
-    <child link="wheel1"/>
-    <origin rpy="0 0 0" xyz="0 0 -0.055"/>
-    <axis xyz="0 1 0"/>
-  </joint>
-<unit_create base_name="base_wheel2_link" wheel_name="wheel2"/>
-  <joint name="base_joint2" type="continuous">
-    <parent link="base_link"/>
-    <child link="base_wheel2_link"/>
+  <joint name="left_front_wheel_joint" type="continuous">
+    <parent link="left_front_steering"/>
+    <child link="left_front_wheel"/>
+    <origin rpy="0 0 0" xyz="0 0 -0.055"/>
+    <axis xyz="0 1 0"/>
+  </joint>
+<unit_create base_name="left_rear_steering" wheel_name="left_rear_wheel"/>
+  <joint name="left_rear_steering_joint" type="continuous">
+    <parent link="base_link"/>
+    <child link="left_rear_steering"/>
     <origin rpy="0 0 0" xyz="-0.35 0.35 -0.055"/>
     <axis xyz="0 0 1"/>
   </joint>
-  <joint name="wheel2_joint" type="continuous">
-    <parent link="base_wheel2_link"/>
-    <child link="wheel2"/>
-    <origin rpy="0 0 0" xyz="0 0 -0.055"/>
-    <axis xyz="0 1 0"/>
-  </joint>
-<unit_create base_name="base_wheel3_link" wheel_name="wheel3"/>
-  <joint name="base_joint3" type="continuous">
-    <parent link="base_link"/>
-    <child link="base_wheel3_link"/>
+  <joint name="left_rear_wheel_joint" type="continuous">
+    <parent link="left_rear_steering"/>
+    <child link="left_rear_wheel"/>
+    <origin rpy="0 0 0" xyz="0 0 -0.055"/>
+    <axis xyz="0 1 0"/>
+  </joint>
+<unit_create base_name="right_front_steering" wheel_name="right_front_wheel"/>
+  <joint name="right_front_steering_joint" type="continuous">
+    <parent link="base_link"/>
+    <child link="right_front_steering"/>
     <origin rpy="0 0 0" xyz="0.35 -0.35 -0.055"/>
     <axis xyz="0 0 1"/>
   </joint>
-  <joint name="wheel3_joint" type="continuous">
-    <parent link="base_wheel3_link"/>
-    <child link="wheel3"/>
-    <origin rpy="0 0 0" xyz="0 0 -0.055"/>
-    <axis xyz="0 1 0"/>
-  </joint>
-<unit_create base_name="base_wheel4_link" wheel_name="wheel4"/>
-  <joint name="base_joint4" type="continuous">
-    <parent link="base_link"/>
-    <child link="base_wheel4_link"/>
+  <joint name="right_front_wheel_joint" type="continuous">
+    <parent link="right_front_steering"/>
+    <child link="right_front_wheel"/>
+    <origin rpy="0 0 0" xyz="0 0 -0.055"/>
+    <axis xyz="0 1 0"/>
+  </joint>
+<unit_create base_name="right_rear_steering" wheel_name="right_rear_wheel"/>
+  <joint name="right_rear_steering_joint" type="continuous">
+    <parent link="base_link"/>
+    <child link="right_rear_steering"/>
     <origin rpy="0 0 0" xyz="-0.35 -0.35 -0.055"/>
     <axis xyz="0 0 1"/>
   </joint>
-  <joint name="wheel4_joint" type="continuous">
-    <parent link="base_wheel4_link"/>
-    <child link="wheel4"/>
+  <joint name="right_rear_wheel_joint" type="continuous">
+    <parent link="right_rear_steering"/>
+    <child link="right_rear_wheel"/>
     <origin rpy="0 0 0" xyz="0 0 -0.055"/>
     <axis xyz="0 1 0"/>
@@ -66,5 +66,5 @@
  </joint>
   <!-- Hokuyo Laser -->
-  <link name="hokuyo_link">
+  <link name="left_hokuyo_link">
     <collision>
       <origin xyz="0 0 0" rpy="0 0 0"/>
@@ -80,72 +80,36 @@
     </visual>
   </link>
-  <joint name="hokuyo_joint" type="fixed">
+  <joint name="left_hokuyo_joint" type="fixed">
     <axis xyz="0 1 0" />
-    <origin xyz="0 0.4 0.1" rpy="0 0 1.5"/>
-    <parent link="base_link"/>
-    <child link="hokuyo_link"/>
-  </joint>
-<link name="marker1">
+    <origin xyz="0.4 0.4 0.1" rpy="0 0 ${M_PI/4}"/>
+    <parent link="base_link"/>
+    <child link="left_hokuyo_link"/>
+  </joint>
+  <!-- Hokuyo Laser -->
+  <link name="right_hokuyo_link">
+    <collision>
+      <origin xyz="0 0 0" rpy="0 0 0"/>
+      <geometry>
+        <box size="0.1 0.1 0.1"/>
+      </geometry>
+    </collision>
     <visual>
       <origin xyz="0 0 0" rpy="0 0 0"/>
       <geometry>
-        <box size="0.01 0.01 0.01"/>
+        <mesh filename="package://rrbot_description/meshes/hokuyo.dae"/>
       </geometry>
     </visual>
   </link>
-  <joint name="fix1" type="fixed">
-    <origin xyz="0 0 0.3" rpy="0 0 0"/>
-    <parent link="wheel1"/>
-    <child link="marker1"/>
-  </joint>
-<link name="marker2">
-    <visual>
-      <origin xyz="0 0 0" rpy="0 0 0"/>
-      <geometry>
-        <box size="0.01 0.01 0.01"/>
-      </geometry>
-    </visual>
-  </link>
-  <joint name="fix2" type="fixed">
-    <origin xyz="0 0 0.3" rpy="0 0 0"/>
-    <parent link="wheel2"/>
-    <child link="marker2"/>
-  </joint>
-<link name="marker3">
-    <visual>
-      <origin xyz="0 0 0" rpy="0 0 0"/>
-      <geometry>
-        <box size="0.01 0.01 0.01"/>
-      </geometry>
-    </visual>
-  </link>
-  <joint name="fix3" type="fixed">
-    <origin xyz="0 0 0.3" rpy="0 0 0"/>
-    <parent link="wheel3"/>
-    <child link="marker3"/>
-  </joint>
-<link name="marker4">
-    <visual>
-      <origin xyz="0 0 0" rpy="0 0 0"/>
-      <geometry>
-        <box size="0.01 0.01 0.01"/>
-      </geometry>
-    </visual>
-    <inertial>
-      <mass value="1e-5" />
-      <origin xyz="0 0 0" rpy="0 0 0"/>
-      <inertia ixx="1e-6" ixy="0" ixz="0" iyy="1e-6" iyz="0" izz="1e-6" />
-    </inertial>
-  </link>
-  <joint name="fix4" type="fixed">
-    <origin xyz="0 0 0.3" rpy="0 0 0"/>
-    <parent link="wheel4"/>
-    <child link="marker4"/>
+  <joint name="right_hokuyo_joint" type="fixed">
+    <axis xyz="0 1 0" />
+    <origin xyz="-0.4 -0.4 0.1" rpy="0 0 ${-3*M_PI/4}"/>
+    <parent link="base_link"/>
+    <child link="right_hokuyo_link"/>
   </joint>
   <!-- ===============  Transmission ===============-->
- <trans_create base_joint_name="base_joint1" wheel_name="wheel1"/>
-<trans_create base_joint_name="base_joint2" wheel_name="wheel2"/>
-<trans_create base_joint_name="base_joint3" wheel_name="wheel3"/>
-<trans_create base_joint_name="base_joint4" wheel_name="wheel4"/>
+ <trans_create base_joint_name="left_front_steering_joint" wheel_name="left_front_wheel"/>
+<trans_create base_joint_name="left_rear_steering_joint" wheel_name="left_rear_wheel"/>
+<trans_create base_joint_name="right_front_steering_joint" wheel_name="right_front_wheel"/>
+<trans_create base_joint_name="right_rear_steering_joint" wheel_name="right_rear_wheel"/>
   <!-- =============== Gazebo =============== -->
   <gazebo>
@@ -159,5 +123,5 @@
     <mu2 value="${mu}" />
   </gazebo>
- <gazebo reference="base_wheel1_link">
+ <gazebo reference="left_front_steering">
    <selfCollide>true</selfCollide>
      <!-- This caster is no frictional resistance. -->
@@ -165,29 +129,29 @@
     <mu2 value="${mu}" />
   </gazebo>
-<gazebo reference="wheel1">
-   <selfCollide>true</selfCollide>
-     <!-- This caster is no frictional resistance. -->
-    <mu1 value="${mu}" />
-    <mu2 value="${mu}" />
-  </gazebo>
- <gazebo reference="base_wheel2_link">
-   <selfCollide>true</selfCollide>
-     <!-- This caster is no frictional resistance. -->
-    <mu1 value="${mu}" />
-    <mu2 value="${mu}" />
-  </gazebo>
-<gazebo reference="wheel2">
-   <selfCollide>true</selfCollide>
-     <!-- This caster is no frictional resistance. -->
-    <mu1 value="${mu}" />
-    <mu2 value="${mu}" />
-  </gazebo>
- <gazebo reference="base_wheel3_link">
-   <selfCollide>true</selfCollide>
-     <!-- This caster is no frictional resistance. -->
-    <mu1 value="${mu}" />
-    <mu2 value="${mu}" />
-  </gazebo>
-<gazebo reference="wheel3">
+<gazebo reference="left_front_wheel">
+   <selfCollide>true</selfCollide>
+     <!-- This caster is no frictional resistance. -->
+    <mu1 value="${mu}" />
+    <mu2 value="${mu}" />
+  </gazebo>
+ <gazebo reference="left_rear_steering">
+   <selfCollide>true</selfCollide>
+     <!-- This caster is no frictional resistance. -->
+    <mu1 value="${mu}" />
+    <mu2 value="${mu}" />
+  </gazebo>
+<gazebo reference="left_rear_wheel">
+   <selfCollide>true</selfCollide>
+     <!-- This caster is no frictional resistance. -->
+    <mu1 value="${mu}" />
+    <mu2 value="${mu}" />
+  </gazebo>
+ <gazebo reference="right_front_steering">
+   <selfCollide>true</selfCollide>
+     <!-- This caster is no frictional resistance. -->
+    <mu1 value="${mu}" />
+    <mu2 value="${mu}" />
+  </gazebo>
+<gazebo reference="right_front_wheel">
    <selfCollide>true</selfCollide>
      <!-- This caster is no frictional resistance. -->
@@ -195,11 +159,11 @@
     <mu2 value="${mu}" />
 </gazebo>
- <gazebo reference="base_wheel4_link">
-   <selfCollide>true</selfCollide>
-     <!-- This caster is no frictional resistance. -->
-    <mu1 value="${mu}" />
-    <mu2 value="${mu}" />
-  </gazebo>
-<gazebo reference="wheel4">
+ <gazebo reference="right_rear_steering">
+   <selfCollide>true</selfCollide>
+     <!-- This caster is no frictional resistance. -->
+    <mu1 value="${mu}" />
+    <mu2 value="${mu}" />
+  </gazebo>
+<gazebo reference="right_rear_wheel">
    <selfCollide>true</selfCollide>
      <!-- This caster is no frictional resistance. -->
@@ -208,6 +172,6 @@
   </gazebo>
   <!-- hokuyo -->
-  <gazebo reference="hokuyo_link">
-    <sensor type="ray" name="head_hokuyo_sensor">
+  <gazebo reference="left_hokuyo_link">
+    <sensor type="ray" name="left_hokuyo_sensor">
       <pose>0 0 0 0 0 0</pose>
       <visualize>false</visualize>
@@ -237,9 +201,45 @@
         </noise>
       </ray>
-      <plugin name="gazebo_ros_head_hokuyo_controller" filename="libgazebo_ros_laser.so">
-        <topicName>/rrbot/laser/scan</topicName>
-        <frameName>hokuyo_link</frameName>
+      <plugin name="gazebo_ros_left_hokuyo_controller" filename="libgazebo_ros_laser.so">
+        <topicName>/rrbot/laser/left_scan</topicName>
+        <frameName>left_hokuyo_link</frameName>
       </plugin>
     </sensor>
   </gazebo>
+  <!-- hokuyo -->
+  <gazebo reference="right_hokuyo_link">
+    <sensor type="ray" name="right_hokuyo_sensor">
+      <pose>0 0 0 0 0 0</pose>
+      <visualize>false</visualize>
+      <update_rate>40</update_rate>
+      <ray>
+        <scan>
+          <horizontal>
+            <samples>720</samples>
+            <resolution>1</resolution>
+            <min_angle>-1.570796</min_angle>
+            <max_angle>1.570796</max_angle>
+          </horizontal>
+        </scan>
+        <range>
+          <min>0.10</min>
+          <max>30.0</max>
+          <resolution>0.01</resolution>
+        </range>
+        <noise>
+          <type>gaussian</type>
+          <!-- Noise parameters based on published spec for Hokuyo laser
+               achieving "+-30mm" accuracy at range < 10m.  A mean of 0.0m and
+               stddev of 0.01m will put 99.7% of samples within 0.03m of the true
+               reading. -->
+          <mean>0.0</mean>
+          <stddev>0.01</stddev>
+        </noise>
+      </ray>
+      <plugin name="gazebo_ros_right_hokuyo_controller" filename="libgazebo_ros_laser.so">
+        <topicName>/rrbot/laser/right_scan</topicName>
+        <frameName>right_hokuyo_link</frameName>
+      </plugin>
+    </sensor>
+  </gazebo>
 </robot>

Commit message: model change

File: src/simc/urdf/common.xacro (robot description, xacro)
@@ -22,5 +22,5 @@
     <collision>
       <geometry>
-        <box size="${width} ${depth} ${height}"/>
+      <box size="${width} ${depth} ${height}"/>
       </geometry>
     </collision>
@@ -50,8 +50,8 @@
 <xacro:macro name="unit_create" params="base_name wheel_name">
 	<link name="${base_name}">
-    <cylinder_create rpy="0" mass="0.1" radius="0.05" length="0.01"/>
+    <cylinder_create rpy="0" mass="0.1" radius="0.05" length="0.004"/>
   </link>
   <link name="${wheel_name}">
-    <cylinder_create rpy="${M_PI/2}" mass="0.1" radius="0.05" length="0.05"/>
+    <cylinder_create rpy="${M_PI/2}" mass="0.1" radius="0.05" length="0.01"/>
   </link>
   </xacro:macro>

File: src/simc/urdf/my_robo.xacro (robot description, xacro)
@@ -5,5 +5,5 @@
 <xacro:property name="mu" value="0.5"/>
  <link name="base_link">
-    <box_create mass="10" height="0.1" width="0.8" depth="0.8"/>
+    <box_create mass="30" height="0.004" width="0.877" depth="0.877"/>
  </link>
 <unit_create base_name="base_wheel1_link" wheel_name="wheel1"/>
@@ -11,5 +11,5 @@
     <parent link="base_link"/>
     <child link="base_wheel1_link"/>
-    <origin rpy="0 0 0" xyz="0.35 0.35 -0.055"/>
+    <origin rpy="0 0 0" xyz="0.265 0.265 0"/>
     <axis xyz="0 0 1"/>
   </joint>
@@ -17,5 +17,5 @@
     <parent link="base_wheel1_link"/>
     <child link="wheel1"/>
-    <origin rpy="0 0 0" xyz="0 0 -0.055"/>
+    <origin rpy="0 0 0" xyz="0 0 0.028"/>
     <axis xyz="0 1 0"/>
   </joint>
@@ -24,5 +24,5 @@
     <parent link="base_link"/>
     <child link="base_wheel2_link"/>
-    <origin rpy="0 0 0" xyz="-0.35 0.35 -0.055"/>
+    <origin rpy="0 0 0" xyz="-0.265 0.265 0"/>
     <axis xyz="0 0 1"/>
   </joint>
@@ -30,5 +30,5 @@
     <parent link="base_wheel2_link"/>
     <child link="wheel2"/>
-    <origin rpy="0 0 0" xyz="0 0 -0.055"/>
+    <origin rpy="0 0 0" xyz="0 0 0.028"/>
     <axis xyz="0 1 0"/>
   </joint>
@@ -37,5 +37,5 @@
     <parent link="base_link"/>
     <child link="base_wheel3_link"/>
-    <origin rpy="0 0 0" xyz="0.35 -0.35 -0.055"/>
+    <origin rpy="0 0 0" xyz="-0.265 -0.265 0"/>
     <axis xyz="0 0 1"/>
   </joint>
@@ -43,5 +43,5 @@
     <parent link="base_wheel3_link"/>
     <child link="wheel3"/>
-    <origin rpy="0 0 0" xyz="0 0 -0.055"/>
+    <origin rpy="0 0 0" xyz="0 0 0.028"/>
     <axis xyz="0 1 0"/>
   </joint>
@@ -50,5 +50,5 @@
     <parent link="base_link"/>
     <child link="base_wheel4_link"/>
-    <origin rpy="0 0 0" xyz="-0.35 -0.35 -0.055"/>
+    <origin rpy="0 0 0" xyz="0.265 -0.265 0"/>
     <axis xyz="0 0 1"/>
   </joint>
@@ -56,15 +56,15 @@
     <parent link="base_wheel4_link"/>
     <child link="wheel4"/>
-    <origin rpy="0 0 0" xyz="0 0 -0.055"/>
-    <axis xyz="0 1 0"/>
-  </joint>
+    <origin rpy="0 0 0" xyz="0 0 0.028"/>
+    <axis xyz="0 1 0"/>
+  </joint>-->
 <link name="base_footprint"/>
   <joint name="base_joint" type="fixed">
    <parent link="base_footprint"/>
    <child link="base_link"/>
-   <origin rpy="0 0 0" xyz="0 0 0.16"/>
+   <origin rpy="0 0 0" xyz="0 0 0.022"/>
  </joint>
-  <!-- Hokuyo Laser -->
-  <link name="hokuyo_link">
+Hokuyo Laser
+  <link name="hokuyo_link1">
     <collision>
       <origin xyz="0 0 0" rpy="0 0 0"/>
@@ -80,9 +80,29 @@
     </visual>
   </link>
-  <joint name="hokuyo_joint" type="fixed">
+  <joint name="hokuyo_joint1" type="fixed">
     <axis xyz="0 1 0" />
-    <origin xyz="0 0.4 0.1" rpy="0 0 1.5"/>
-    <parent link="base_link"/>
-    <child link="hokuyo_link"/>
+    <origin xyz="0.4385 -0.4385 0.002" rpy="0 0 ${M_PI*3/4}"/>
+    <parent link="base_link"/>
+    <child link="hokuyo_link1"/>
+  </joint>
+  <link name="hokuyo_link2">
+    <collision>
+      <origin xyz="0 0 0" rpy="0 0 0"/>
+      <geometry>
+        <box size="0.1 0.1 0.1"/>
+      </geometry>
+    </collision>
+    <visual>
+      <origin xyz="0 0 0" rpy="0 0 0"/>
+      <geometry>
+        <mesh filename="package://rrbot_description/meshes/hokuyo.dae"/>
+      </geometry>
+    </visual>
+  </link>
+  <joint name="hokuyo_joint2" type="fixed">
+    <axis xyz="0 1 0" />
+    <origin xyz="-0.4385 0.4385 0.002" rpy="0 0 ${-M_PI/4}"/>
+    <parent link="base_link"/>
+    <child link="hokuyo_link2"/>
   </joint>
 <link name="marker1">
@@ -144,5 +164,5 @@
   </joint>
   <!-- ===============  Transmission ===============-->
- <trans_create base_joint_name="base_joint1" wheel_name="wheel1"/>
+<trans_create base_joint_name="base_joint1" wheel_name="wheel1"/>
 <trans_create base_joint_name="base_joint2" wheel_name="wheel2"/>
 <trans_create base_joint_name="base_joint3" wheel_name="wheel3"/>
@@ -161,5 +181,4 @@
  <gazebo reference="base_wheel1_link">
    <selfCollide>true</selfCollide>
-     <!-- This caster is no frictional resistance. -->
       <mu1 value="${mu}" />
     <mu2 value="${mu}" />
@@ -167,11 +186,9 @@
 <gazebo reference="wheel1">
    <selfCollide>true</selfCollide>
-     <!-- This caster is no frictional resistance. -->
-    <mu1 value="${mu}" />
-    <mu2 value="${mu}" />
-  </gazebo>
- <gazebo reference="base_wheel2_link">
-   <selfCollide>true</selfCollide>
-     <!-- This caster is no frictional resistance. -->
+    <mu1 value="${mu}" />
+    <mu2 value="${mu}" />
+  </gazebo>
+  <gazebo reference="base_wheel2_link">
+   <selfCollide>true</selfCollide>
     <mu1 value="${mu}" />
     <mu2 value="${mu}" />
@@ -179,5 +196,4 @@
 <gazebo reference="wheel2">
    <selfCollide>true</selfCollide>
-     <!-- This caster is no frictional resistance. -->
     <mu1 value="${mu}" />
     <mu2 value="${mu}" />
@@ -185,5 +201,4 @@
  <gazebo reference="base_wheel3_link">
    <selfCollide>true</selfCollide>
-     <!-- This caster is no frictional resistance. -->
     <mu1 value="${mu}" />
     <mu2 value="${mu}" />
@@ -191,5 +206,4 @@
 <gazebo reference="wheel3">
    <selfCollide>true</selfCollide>
-     <!-- This caster is no frictional resistance. -->
     <mu1 value="${mu}" />
     <mu2 value="${mu}" />
@@ -197,5 +211,4 @@
  <gazebo reference="base_wheel4_link">
    <selfCollide>true</selfCollide>
-     <!-- This caster is no frictional resistance. -->
     <mu1 value="${mu}" />
     <mu2 value="${mu}" />
@@ -203,10 +216,9 @@
 <gazebo reference="wheel4">
    <selfCollide>true</selfCollide>
-     <!-- This caster is no frictional resistance. -->
-    <mu1 value="${mu}" />
-    <mu2 value="${mu}" />
-  </gazebo>
-  <!-- hokuyo -->
-  <gazebo reference="hokuyo_link">
+    <mu1 value="${mu}" />
+    <mu2 value="${mu}" />
+  </gazebo>
+  <!-- hokuyo-->
+  <gazebo reference="hokuyo_link1">
     <sensor type="ray" name="head_hokuyo_sensor">
       <pose>0 0 0 0 0 0</pose>
@@ -229,5 +241,5 @@
         <noise>
           <type>gaussian</type>
-          <!-- Noise parameters based on published spec for Hokuyo laser
+          <!--Noise parameters based on published spec for Hokuyo laser
                achieving "+-30mm" accuracy at range < 10m.  A mean of 0.0m and
                stddev of 0.01m will put 99.7% of samples within 0.03m of the true
@@ -238,8 +250,43 @@
       </ray>
       <plugin name="gazebo_ros_head_hokuyo_controller" filename="libgazebo_ros_laser.so">
-        <topicName>/rrbot/laser/scan</topicName>
-        <frameName>hokuyo_link</frameName>
+        <topicName>/rrbot/laser/scan1</topicName>
+        <frameName>hokuyo_link1</frameName>
       </plugin>
     </sensor>
   </gazebo>
+  <gazebo reference="hokuyo_link2">
+    <sensor type="ray" name="head_hokuyo_sensor">
+      <pose>0 0 0 0 0 0</pose>
+      <visualize>false</visualize>
+      <update_rate>40</update_rate>
+      <ray>
+        <scan>
+          <horizontal>
+            <samples>720</samples>
+            <resolution>1</resolution>
+            <min_angle>-1.570796</min_angle>
+            <max_angle>1.570796</max_angle>
+          </horizontal>
+        </scan>
+        <range>
+          <min>0.10</min>
+          <max>30.0</max>
+          <resolution>0.01</resolution>
+        </range>
+        <noise>
+          <type>gaussian</type>
+         <!-- Noise parameters based on published spec for Hokuyo laser
+               achieving "+-30mm" accuracy at range < 10m.  A mean of 0.0m and
+               stddev of 0.01m will put 99.7% of samples within 0.03m of the true
+               reading. -->
+          <mean>0.0</mean>
+          <stddev>0.01</stddev>
+        </noise>
+      </ray>
+      <plugin name="gazebo_ros_head_hokuyo_controller" filename="libgazebo_ros_laser.so">
+        <topicName>/rrbot/laser/scan2</topicName>
+        <frameName>hokuyo_link2</frameName>
+      </plugin>
+    </sensor>
+  </gazebo>
 </robot>
