Commit message: パラメータを変えたモデル

File: src/simc/urdf/common.xacro (robot description, xacro)
@@ -22,5 +22,5 @@
     <collision>
       <geometry>
-        <box size="${width} ${depth} ${height}"/>
+      <box size="${width} ${depth} ${height}"/>
       </geometry>
     </collision>
@@ -50,8 +50,8 @@
 <xacro:macro name="unit_create" params="base_name wheel_name">
 	<link name="${base_name}">
-    <cylinder_create rpy="0" mass="0.1" radius="0.05" length="0.01"/>
+    <cylinder_create rpy="0" mass="0.1" radius="0.05" length="0.004"/>
   </link>
   <link name="${wheel_name}">
-    <cylinder_create rpy="${M_PI/2}" mass="0.1" radius="0.05" length="0.05"/>
+    <cylinder_create rpy="${M_PI/2}" mass="0.1" radius="0.05" length="0.01"/>
   </link>
   </xacro:macro>
@@ -60,8 +60,8 @@
       <type>transmission_interface/SimpleTransmission</type>
       <joint name="${base_joint_name}">
-  <hardwareInterface>hardware_interface/PositionJointInterface</hardwareInterface>
+  <hardwareInterface>PositionJointInterface</hardwareInterface>
       </joint>
    <actuator name="${base_joint_name}_motor">
-  <hardwareInterface>hardware_interface/PositionJointInterface</hardwareInterface>
+  <hardwareInterface>PositionJointInterface</hardwareInterface>
   <mechanicalReduction>100</mechanicalReduction>
       </actuator>
@@ -70,8 +70,8 @@
       <type>transmission_interface/SimpleTransmission</type>
       <joint name="${wheel_name}_joint">
-  <hardwareInterface>hardware_interface/VelocityJointInterface</hardwareInterface>
+  <hardwareInterface>VelocityJointInterface</hardwareInterface>
       </joint>
    <actuator name="${wheel_name}_motor">
-  <hardwareInterface>hardware_interface/VelocityJointInterface</hardwareInterface>
+  <hardwareInterface>VelocityJointInterface</hardwareInterface>
   <mechanicalReduction>100</mechanicalReduction>
       </actuator>

File: src/simc/urdf/my_robo.xacro (robot description, xacro)
@@ -5,5 +5,5 @@
 <xacro:property name="mu" value="0.5"/>
  <link name="base_link">
-    <box_create mass="10" height="0.1" width="0.8" depth="0.8"/>
+    <box_create mass="30" height="0.004" width="0.877" depth="0.877"/>
  </link>
 <unit_create base_name="left_front_steering" wheel_name="left_front_wheel"/>
@@ -11,5 +11,5 @@
     <parent link="base_link"/>
     <child link="left_front_steering"/>
-    <origin rpy="0 0 0" xyz="0.35 0.35 -0.055"/>
+    <origin rpy="0 0 0" xyz="0.265 0.265 0"/>
     <axis xyz="0 0 1"/>
   </joint>
@@ -17,5 +17,5 @@
     <parent link="left_front_steering"/>
     <child link="left_front_wheel"/>
-    <origin rpy="0 0 0" xyz="0 0 -0.055"/>
+    <origin rpy="0 0 0" xyz="0 0 0.028"/>
     <axis xyz="0 1 0"/>
   </joint>
@@ -24,5 +24,5 @@
     <parent link="base_link"/>
     <child link="left_rear_steering"/>
-    <origin rpy="0 0 0" xyz="-0.35 0.35 -0.055"/>
+    <origin rpy="0 0 0" xyz="-0.265 0.265 0"/>
     <axis xyz="0 0 1"/>
   </joint>
@@ -30,5 +30,5 @@
     <parent link="left_rear_steering"/>
     <child link="left_rear_wheel"/>
-    <origin rpy="0 0 0" xyz="0 0 -0.055"/>
+    <origin rpy="0 0 0" xyz="0 0 0.028"/>
     <axis xyz="0 1 0"/>
   </joint>
@@ -37,5 +37,5 @@
     <parent link="base_link"/>
     <child link="right_front_steering"/>
-    <origin rpy="0 0 0" xyz="0.35 -0.35 -0.055"/>
+    <origin rpy="0 0 0" xyz="-0.265 -0.265 0"/>
     <axis xyz="0 0 1"/>
   </joint>
@@ -43,5 +43,5 @@
     <parent link="right_front_steering"/>
     <child link="right_front_wheel"/>
-    <origin rpy="0 0 0" xyz="0 0 -0.055"/>
+    <origin rpy="0 0 0" xyz="0 0 0.028"/>
     <axis xyz="0 1 0"/>
   </joint>
@@ -50,5 +50,5 @@
     <parent link="base_link"/>
     <child link="right_rear_steering"/>
-    <origin rpy="0 0 0" xyz="-0.35 -0.35 -0.055"/>
+    <origin rpy="0 0 0" xyz="0.265 -0.265 0"/>
     <axis xyz="0 0 1"/>
   </joint>
@@ -56,5 +56,5 @@
     <parent link="right_rear_steering"/>
     <child link="right_rear_wheel"/>
-    <origin rpy="0 0 0" xyz="0 0 -0.055"/>
+    <origin rpy="0 0 0" xyz="0 0 0.028"/>
     <axis xyz="0 1 0"/>
   </joint>
@@ -63,8 +63,7 @@
    <parent link="base_footprint"/>
    <child link="base_link"/>
-   <origin rpy="0 0 0" xyz="0 0 0.16"/>
+   <origin rpy="0 0 0" xyz="0 0 0.022"/>
  </joint>
-  <!-- Hokuyo Laser -->
-  <link name="left_hokuyo_link">
+ <link name="left_hokuyo_link">
     <collision>
       <origin xyz="0 0 0" rpy="0 0 0"/>
@@ -82,10 +81,9 @@
   <joint name="left_hokuyo_joint" type="fixed">
     <axis xyz="0 1 0" />
-    <origin xyz="0.4 0.4 0.1" rpy="0 0 ${M_PI/4}"/>
+    <origin xyz="0.4385 -0.4385 0.002" rpy="0 0 ${M_PI*3/4}"/>
     <parent link="base_link"/>
     <child link="left_hokuyo_link"/>
   </joint>
-  <!-- Hokuyo Laser -->
-  <link name="right_hokuyo_link">
+<link name="right_hokuyo_link">
     <collision>
       <origin xyz="0 0 0" rpy="0 0 0"/>
@@ -103,8 +101,66 @@
   <joint name="right_hokuyo_joint" type="fixed">
     <axis xyz="0 1 0" />
-    <origin xyz="-0.4 -0.4 0.1" rpy="0 0 ${-3*M_PI/4}"/>
+    <origin xyz="-0.4385 0.4385 0.002" rpy="0 0 ${-M_PI/4}"/>
     <parent link="base_link"/>
     <child link="right_hokuyo_link"/>
   </joint>
+<!--
+<link name="marker1">
+    <visual>
+      <origin xyz="0 0 0" rpy="0 0 0"/>
+      <geometry>
+        <box size="0.01 0.01 0.01"/>
+      </geometry>
+    </visual>
+  </link>
+  <joint name="fix1" type="fixed">
+    <origin xyz="0 0 0.3" rpy="0 0 0"/>
+    <parent link="wheel1"/>
+    <child link="marker1"/>
+  </joint>
+<link name="marker2">
+    <visual>
+      <origin xyz="0 0 0" rpy="0 0 0"/>
+      <geometry>
+        <box size="0.01 0.01 0.01"/>
+      </geometry>
+    </visual>
+  </link>
+  <joint name="fix2" type="fixed">
+    <origin xyz="0 0 0.3" rpy="0 0 0"/>
+    <parent link="wheel2"/>
+    <child link="marker2"/>
+  </joint>
+<link name="marker3">
+    <visual>
+      <origin xyz="0 0 0" rpy="0 0 0"/>
+      <geometry>
+        <box size="0.01 0.01 0.01"/>
+      </geometry>
+    </visual>
+  </link>
+  <joint name="fix3" type="fixed">
+    <origin xyz="0 0 0.3" rpy="0 0 0"/>
+    <parent link="wheel3"/>
+    <child link="marker3"/>
+  </joint>
+<link name="marker4">
+    <visual>
+      <origin xyz="0 0 0" rpy="0 0 0"/>
+      <geometry>
+        <box size="0.01 0.01 0.01"/>
+      </geometry>
+    </visual>
+    <inertial>
+      <mass value="1e-5" />
+      <origin xyz="0 0 0" rpy="0 0 0"/>
+      <inertia ixx="1e-6" ixy="0" ixz="0" iyy="1e-6" iyz="0" izz="1e-6" />
+    </inertial>
+  </link>
+  <joint name="fix4" type="fixed">
+    <origin xyz="0 0 0.3" rpy="0 0 0"/>
+    <parent link="wheel4"/>
+    <child link="marker4"/>
+  </joint>-->
   <!-- ===============  Transmission ===============-->
  <trans_create base_joint_name="left_front_steering_joint" wheel_name="left_front_wheel"/>
@@ -112,5 +168,5 @@
 <trans_create base_joint_name="right_front_steering_joint" wheel_name="right_front_wheel"/>
 <trans_create base_joint_name="right_rear_steering_joint" wheel_name="right_rear_wheel"/>
-  <!-- =============== Gazebo =============== -->
+   <!-- =============== Gazebo =============== -->
   <gazebo>
     <plugin name="gazebo_ros_control" filename="libgazebo_ros_control.so">
