Commit message: 多分実際に動く

File: src/simc/urdf/my_robo.xacro (robot description, xacro)
@@ -11,5 +11,5 @@
     <parent link="base_link"/>
     <child link="left_front_steering"/>
-    <origin rpy="0 0 0" xyz="0.265 0.265 0"/>
+    <origin rpy="0 0 ${3*M_PI/4}" xyz="0.265 0.265 0"/>
     <axis xyz="0 0 1"/>
   </joint>
@@ -24,5 +24,5 @@
     <parent link="base_link"/>
     <child link="left_rear_steering"/>
-    <origin rpy="0 0 0" xyz="-0.265 0.265 0"/>
+    <origin rpy="0 0 ${-3*M_PI/4}" xyz="-0.265 0.265 0"/>
     <axis xyz="0 0 1"/>
   </joint>
@@ -33,9 +33,22 @@
     <axis xyz="0 1 0"/>
   </joint>
+<unit_create base_name="right_rear_steering" wheel_name="right_rear_wheel"/>
+  <joint name="right_rear_steering_joint" type="continuous">
+    <parent link="base_link"/>
+    <child link="right_rear_steering"/>
+    <origin rpy="0 0 ${-M_PI/4}" xyz="-0.265 -0.265 0"/>
+    <axis xyz="0 0 1"/>
+  </joint>
+  <joint name="right_rear_wheel_joint" type="continuous">
+    <parent link="right_rear_steering"/>
+    <child link="right_rear_wheel"/>
+    <origin rpy="0 0 0" xyz="0 0 0.028"/>
+    <axis xyz="0 1 0"/>
+  </joint>
 <unit_create base_name="right_front_steering" wheel_name="right_front_wheel"/>
   <joint name="right_front_steering_joint" type="continuous">
     <parent link="base_link"/>
     <child link="right_front_steering"/>
-    <origin rpy="0 0 0" xyz="-0.265 -0.265 0"/>
+    <origin rpy="0 0 ${M_PI/4}" xyz="0.265 -0.265 0"/>
     <axis xyz="0 0 1"/>
   </joint>
@@ -43,17 +56,4 @@
     <parent link="right_front_steering"/>
     <child link="right_front_wheel"/>
-    <origin rpy="0 0 0" xyz="0 0 0.028"/>
-    <axis xyz="0 1 0"/>
-  </joint>
-<unit_create base_name="right_rear_steering" wheel_name="right_rear_wheel"/>
-  <joint name="right_rear_steering_joint" type="continuous">
-    <parent link="base_link"/>
-    <child link="right_rear_steering"/>
-    <origin rpy="0 0 0" xyz="0.265 -0.265 0"/>
-    <axis xyz="0 0 1"/>
-  </joint>
-  <joint name="right_rear_wheel_joint" type="continuous">
-    <parent link="right_rear_steering"/>
-    <child link="right_rear_wheel"/>
     <origin rpy="0 0 0" xyz="0 0 0.028"/>
     <axis xyz="0 1 0"/>
@@ -81,5 +81,5 @@
   <joint name="left_hokuyo_joint" type="fixed">
     <axis xyz="0 1 0" />
-    <origin xyz="0.4385 -0.4385 0.002" rpy="0 0 ${M_PI*3/4}"/>
+    <origin xyz="0.4385 0.4385 0.002" rpy="0 0 ${M_PI*3/4}"/>
     <parent link="base_link"/>
     <child link="left_hokuyo_link"/>
@@ -101,5 +101,5 @@
   <joint name="right_hokuyo_joint" type="fixed">
     <axis xyz="0 1 0" />
-    <origin xyz="-0.4385 0.4385 0.002" rpy="0 0 ${-M_PI/4}"/>
+    <origin xyz="-0.4385 -0.4385 0.002" rpy="0 0 ${-M_PI/4}"/>
     <parent link="base_link"/>
     <child link="right_hokuyo_link"/>
@@ -166,6 +166,6 @@
  <trans_create base_joint_name="left_front_steering_joint" wheel_name="left_front_wheel"/>
 <trans_create base_joint_name="left_rear_steering_joint" wheel_name="left_rear_wheel"/>
+<trans_create base_joint_name="right_rear_steering_joint" wheel_name="right_rear_wheel"/>
 <trans_create base_joint_name="right_front_steering_joint" wheel_name="right_front_wheel"/>
-<trans_create base_joint_name="right_rear_steering_joint" wheel_name="right_rear_wheel"/>
    <!-- =============== Gazebo =============== -->
   <gazebo>
@@ -203,4 +203,16 @@
     <mu2 value="${mu}" />
   </gazebo>
+ <gazebo reference="right_rear_steering">
+   <selfCollide>true</selfCollide>
+     <!-- This caster is no frictional resistance. -->
+    <mu1 value="${mu}" />
+    <mu2 value="${mu}" />
+  </gazebo>
+<gazebo reference="right_rear_wheel">
+   <selfCollide>true</selfCollide>
+     <!-- This caster is no frictional resistance. -->
+    <mu1 value="${mu}" />
+    <mu2 value="${mu}" />
+</gazebo>
  <gazebo reference="right_front_steering">
    <selfCollide>true</selfCollide>
@@ -210,16 +222,4 @@
   </gazebo>
 <gazebo reference="right_front_wheel">
-   <selfCollide>true</selfCollide>
-     <!-- This caster is no frictional resistance. -->
-    <mu1 value="${mu}" />
-    <mu2 value="${mu}" />
-</gazebo>
- <gazebo reference="right_rear_steering">
-   <selfCollide>true</selfCollide>
-     <!-- This caster is no frictional resistance. -->
-    <mu1 value="${mu}" />
-    <mu2 value="${mu}" />
-  </gazebo>
-<gazebo reference="right_rear_wheel">
    <selfCollide>true</selfCollide>
      <!-- This caster is no frictional resistance. -->
